File: KiCadDemo/Demo/Demo.kicad_sch (KiCad schematic)
At the start: 0 parts

Commit message: Add files via upload
Check2 schematics
Other:
- added sheet comm (comm.kicad_sch)
- added sheet mcu (mcu.kicad_sch)
- added sheet onewire (onewire.kicad_sch)
- added sheet outputs (outputs.kicad_sch)
- added sheet usb-debug (usb-debug.kicad_sch)
Changed lines of the file:
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@@
 (kicad_sch (version 20230121) (generator eeschema)
   (paper "A4")
-  (sheet (at 41.91 41.91) (size 67.31 41.91) (fields_autoplaced)
+  (sheet (at 143.51 78.74) (size 78.74 43.18) (fields_autoplaced)
     (stroke (width 0.1524) (type solid))
     (fill (color 0 0 0 0.0000))
-    (property "Sheetname" "supply" (at 41.91 41.1984 0)
+    (property "Sheetname" "comm" (at 143.51 78.0284 0)
       (effects (font (size 1.27 1.27)) (justify left bottom))
     )
-    (property "Sheetfile" "supply.kicad_sch" (at 41.91 84.4046 0)
+    (property "Sheetfile" "comm.kicad_sch" (at 143.51 122.5046 0)
+      (effects (font (size 1.27 1.27)) (justify left top))
+    )
+    (instances
+      (project "Demo"
+        (path "/6e73ff2b-554f-4e00-b182-1d8d7d5ce0d1" (page "6"))
+      )
+    )
+  )
+  (sheet (at 40.64 133.35) (size 67.31 40.64) (fields_autoplaced)
+    (stroke (width 0.1524) (type solid))
+    (fill (color 0 0 0 0.0000))
+    (property "Sheetname" "onewire" (at 40.64 132.6384 0)
+      (effects (font (size 1.27 1.27)) (justify left bottom))
+    )
+    (property "Sheetfile" "onewire.kicad_sch" (at 40.64 174.5746 0)
+      (effects (font (size 1.27 1.27)) (justify left top))
+    )
+    (instances
+      (project "Demo"
+        (path "/6e73ff2b-554f-4e00-b182-1d8d7d5ce0d1" (page "4"))
+      )
+    )
+  )
+  (sheet (at 144.78 138.43) (size 77.47 19.05) (fields_autoplaced)
+    (stroke (width 0.1524) (type solid))
+    (fill (color 0 0 0 0.0000))
+    (property "Sheetname" "outputs" (at 144.78 137.7184 0)
+      (effects (font (size 1.27 1.27)) (justify left bottom))
+    )
+    (property "Sheetfile" "outputs.kicad_sch" (at 144.78 158.0646 0)
+      (effects (font (size 1.27 1.27)) (justify left top))
+    )
+    (instances
+      (project "Demo"
+        (path "/6e73ff2b-554f-4e00-b182-1d8d7d5ce0d1" (page "7"))
+      )
+    )
+  )
+  (sheet (at 40.64 78.74) (size 67.31 43.18) (fields_autoplaced)
+    (stroke (width 0.1524) (type solid))
+    (fill (color 0 0 0 0.0000))
+    (property "Sheetname" "mcu" (at 40.64 78.0284 0)
+      (effects (font (size 1.27 1.27)) (justify left bottom))
+    )
+    (property "Sheetfile" "mcu.kicad_sch" (at 40.64 122.5046 0)
+      (effects (font (size 1.27 1.27)) (justify left top))
+    )
+    (instances
+      (project "Demo"
+        (path "/6e73ff2b-554f-4e00-b182-1d8d7d5ce0d1" (page "3"))
+      )
+    )
+  )
+  (sheet (at 40.64 26.67) (size 67.31 41.91) (fields_autoplaced)
+    (stroke (width 0.1524) (type solid))
+    (fill (color 0 0 0 0.0000))
+    (property "Sheetname" "supply" (at 40.64 25.9584 0)
+      (effects (font (size 1.27 1.27)) (justify left bottom))
+    )
+    (property "Sheetfile" "supply.kicad_sch" (at 40.64 69.1646 0)
       (effects (font (size 1.27 1.27)) (justify left top))
     )
@@
       )
     )
+  )
+  (sheet (at 143.51 26.67) (size 78.74 41.91) (fields_autoplaced)
+    (stroke (width 0.1524) (type solid))
+    (fill (color 0 0 0 0.0000))
+    (property "Sheetname" "usb-debug" (at 143.51 25.9584 0)
+      (effects (font (size 1.27 1.27)) (justify left bottom))
+    )
+    (property "Sheetfile" "usb-debug.kicad_sch" (at 143.51 69.1646 0)
+      (effects (font (size 1.27 1.27)) (justify left top))
+    )
+    (instances
+      (project "Demo"
+        (path "/6e73ff2b-554f-4e00-b182-1d8d7d5ce0d1" (page "5"))
+      )
+    )
