File: KiCadDemo/Demo/mcu.kicad_sch (KiCad schematic)
At the start: 15 parts, among them SW1 Reset, U3 STM32F103CBT6, X1 8 MHz

Commit message: Add files via upload
Connections:
- net +3V3: now also C5.2, C6.2, C7.2, C9.2, U3.1 (VBAT), U3.24 (VDD), U3.36 (VDD), U3.48 (VDD)
- net NRST: now reaches C12.1, R3.2, SW1.2, U3.7 (NRST)
Other:
- moved on the sheet: C10, C11, C12, C5, C6, C7, C8, C9, LD2, R11, R3, R4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

Commit message: Check #4
Parts:
- SW1: footprint (none) -> Demo:B3F-4000
Changed lines of the file:
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@@
       (effects (font (size 1.27 1.27)) (justify right))
     )
-    (property "Footprint" "" (at 72.39 72.39 0)
+    (property "Footprint" "Demo:B3F-4000" (at 72.39 72.39 0)
       (effects (font (size 1.27 1.27)) hide)
     )
