File: KiCadDemo/Demo/outputs.kicad_sch (KiCad schematic)
At the start: 14 parts, among them J3 22-05-7025, J4 22-05-7025, J5 22-05-7025, U6 74LS06

Commit message: Add files via upload
Connections:
- net FAN2C renamed FAN2_C
Other:
- moved on the sheet: C13, J3, J4, J5, LD4, LD5, LD6, MOV4, MOV5, MOV6, R10, R8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

Commit message: Check #4
Parts:
- J3, J4, J5: footprint (none) -> Demo:IO2
Changed lines of the file:
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@@
       (effects (font (size 1.27 1.27)))
     )
-    (property "Footprint" "" (at 229.87 74.93 0)
+    (property "Footprint" "Demo:IO2" (at 229.87 74.93 0)
       (effects (font (size 1.27 1.27)) hide)
     )
@@
       (effects (font (size 1.27 1.27)) (justify left))
     )
-    (property "Footprint" "" (at 229.87 135.89 0)
+    (property "Footprint" "Demo:IO2" (at 229.87 135.89 0)
       (effects (font (size 1.27 1.27)) hide)
     )
@@
       (effects (font (size 1.27 1.27)) (justify left))
     )
-    (property "Footprint" "" (at 229.87 102.87 0)
-      (effects (font (size 1.27 1.27)) hide)
-    )
+    (property "Footprint" "Demo:IO2" (at 229.87 102.87 0)
+      (effects (font (size 1.27 1.27)) hide)
+    )
