File: KiCadDemo/Demo/supply.kicad_sch (KiCad schematic)
At the start: 13 parts, among them J1 Power, U1 TSR_1-2450, U2 UA78M33

Commit message: Add files via upload
Other:
- moved on the sheet: C1, C2, C3, C4, D1, D2, F1, J1, L1, LD1, R1, U1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

Commit message: Check #4
Parts:
- J1: footprint (none) -> Demo:Power
- L1: footprint (none) -> Demo:tck141
Connections:
- net pwr1: now reaches F1.1, J1.2 (Pin_2)
- net pwr2: now reaches C1.1, F1.2, L1.1
- net pwr5: now reaches C3.1, D1.1 (K), D2.1 (K), U2.1 (IN)
- net pwr4: now reaches D1.2 (A), U1.3 (Vout)
- net pwr3: now reaches C2.1, L1.2, U1.1 (Vin)
Other:
- moved on the sheet: D1, J1
