File: KiCadDemo/Demo/Demo.kicad_pcb (KiCad board)
At the start: 4 copper layers, 100 x 80 mm, 66 parts, among them J1 Power, J2 22-05-7025, J3 22-05-7025, J4 22-05-7025, J5 22-05-7025, J6 Comm, J7 USB_B_Mini, J8 Debug, M1 BSS84, M2 BSS84, SW1 Reset, U1 TSR_1-2450, U2 UA78M33, U3 STM32F103CBT6, U4 DS1822-PAR, U5 MAX3486, U6 74LS06, X1 8 MHz

Commit message: Add files via upload
Changes proposed by Vicente made.
Parts:
- moved MOV3 2.25 mm to (110.8, 80.6)
- moved U2 1.14 mm to (160.6, 72.8), turned to 90 degrees
- moved MOV2 0.93 mm to (103.8, 92.8)
Routing:
- net V_USB: track 78.9 -> 99.0 mm, vias 4 -> 0
- net +3V3: track 54.7 -> 65.6 mm, vias 15 -> 17
- net /supply/pwr5: track 31.1 -> 22.1 mm
- net FAN1_C: track 84.3 -> 89.3 mm
- net FAN2_C: track 78.9 -> 83.8 mm
- net GND: track 95.2 -> 90.6 mm
- net Net-(LD2-A): track 25.7 -> 29.0 mm
- net Net-(J6-Pin_1): track 25.5 -> 27.7 mm
- net Net-(J6-Pin_3): track 25.7 -> 24.8 mm
- net DQ: track 143.5 -> 143.0 mm, vias 6 -> 5
- net Net-(J3-Pin_2): track 79.9 -> 79.6 mm, vias 4 -> 3
- net Net-(J4-Pin_1): track 46.2 -> 46.0 mm, vias 2 -> 1
- net Net-(LD6-K): vias 2 -> 1
- net Net-(LD5-K): vias 2 -> 1
- net Net-(LD4-K): vias 2 -> 1
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